File: 02_ECAD/PS.kicad_sch (KiCad schematic)
At the start: 73 parts, among them J1 B2P3-VH(LF)(SN), J2 B4P-VH(LF)(SN), Q1 IXFH20N100P, SW1 NE18 2A EE 6AMP, U1 UCC28600, U2 CNY17-1, U3 TL431DBZ

Commit message: *Adding Feedback Circuit Simulation.
Parts:
- R18: value 649 -> 1.5k
- R19: value 35.7k -> 35.2k; PN ERJ-PB3B3572V -> TNPW080535K2BEEN
Other:
- note added: "2.5 at 24V"
- note added: "≈10V"
- note removed: "10V"
- note removed: "2.48 at 24V"
Changed lines of the file:
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@@
     (stroke (width 0) (type default) (color 132 0 0 1))
   )
-  (polyline (pts (xy 180.34 184.785) (xy 180.34 180.34))
+  (polyline (pts (xy 180.34 184.785) (xy 180.34 177.8))
     (stroke (width 0) (type default))
   )
@@
     (effects (font (size 3 3) (thickness 0.6) bold) (justify left bottom))
   )
-  (text "2.48 at 24V" (exclude_from_sim no)
+  (text "2.5 at 24V" (exclude_from_sim no)
  (at 201.93 207.645 0)
     (effects (font (size 1.27 1.27)) (justify left bottom))
@@
     (effects (font (size 1.27 1.27) (thickness 0.254) bold (color 255 255 255 1)) (justify right bottom))
   )
-  (text "10V" (exclude_from_sim no)
+  (text "≈10V" (exclude_from_sim no)
  (at 179.705 184.15 90)
     (effects (font (size 1.27 1.27)) (justify left bottom))
@@
       (effects (font (size 1.27 1.27)) (justify left))
     )
-    (property "Value" "649" (at 196.85 184.15 90)
+    (property "Value" "1.5k" (at 196.85 184.15 90)
       (effects (font (size 1.27 1.27)) (justify left))
     )
@@
       (effects (font (size 1.27 1.27)) (justify left))
     )
-    (property "Value" "35.7k" (at 200.66 198.12 0)
+    (property "Value" "35.2k" (at 200.66 198.12 0)
       (effects (font (size 1.27 1.27)) (justify left))
     )
@@
       (effects (font (size 1.27 1.27)) hide)
     )
-    (property "Datasheet" "~" (at 200.66 195.58 0)
-      (effects (font (size 1.27 1.27)) hide)
-    )
-    (property "Description" "" (at 200.66 195.58 0)
-      (effects (font (size 1.27 1.27)) hide)
-    )
-    (property "PN" "ERJ-PB3B3572V" (at 200.66 195.58 0)
-      (effects (font (size 1.27 1.27)) hide)
-    )
+    (property "Datasheet" "TNPW080535K2BEEN" (at 200.66 195.58 0)
+      (effects (font (size 1.27 1.27)) hide)
+    )
+    (property "Description" "TNPW080535K2BEEN" (at 200.66 195.58 0)
+      (effects (font (size 1.27 1.27)) hide)
+    )
+    (property "PN" "TNPW080535K2BEEN" (at 200.66 195.58 0)
+      (effects (font (size 1.27 1.27)) hide)
+    )

Commit message: Update.
Parts:
- D5: PN (none) -> MMSZ5240B
- R18: PN RK73H1JTTDD6490F -> CRG0402F1K5
Changed lines of the file:
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@@
       (effects (font (size 1.27 1.27)) hide)
     )
-    (property "Datasheet" "~" (at 185.42 190.5 90)
-      (effects (font (size 1.27 1.27)) hide)
-    )
-    (property "Description" "" (at 185.42 190.5 0)
+    (property "Datasheet" "MMSZ5240B" (at 185.42 190.5 90)
+      (effects (font (size 1.27 1.27)) hide)
+    )
+    (property "Description" "MMSZ5240B" (at 185.42 190.5 0)
+      (effects (font (size 1.27 1.27)) hide)
+    )
+    (property "PN" "MMSZ5240B" (at 185.42 190.5 0)
       (effects (font (size 1.27 1.27)) hide)
     )
@@
       (effects (font (size 1.27 1.27)) hide)
     )
-    (property "Datasheet" "~" (at 190.5 185.42 0)
-      (effects (font (size 1.27 1.27)) hide)
-    )
-    (property "Description" "" (at 190.5 185.42 0)
-      (effects (font (size 1.27 1.27)) hide)
-    )
-    (property "PN" "RK73H1JTTDD6490F" (at 190.5 185.42 0)
-      (effects (font (size 1.27 1.27)) hide)
-    )
+    (property "Datasheet" "CRG0402F1K5" (at 190.5 185.42 0)
+      (effects (font (size 1.27 1.27)) hide)
+    )
+    (property "Description" "CRG0402F1K5" (at 190.5 185.42 0)
+      (effects (font (size 1.27 1.27)) hide)
+    )
+    (property "PN" "CRG0402F1K5" (at 190.5 185.42 0)
+      (effects (font (size 1.27 1.27)) hide)
+    )
