File: 01_ECAD/ACDC150V24.kicad_pcb (KiCad board)
At the start: 2 copper layers, 85 x 120 mm, 73 parts, among them J1 B2P3-VH(LF)(SN), J2 B4P-VH(LF)(SN), Q1 IXFH20N100P, SW1 NE18 2A EE 6AMP, U1 UCC28600, U2 CNY17-1, U3 TL431DBZ

Commit message: UPDATE!
Parts:
- removed the R1 at (38.0, 86.8)
- removed R22, R23, R24, R25, R26: 20K, Resistor_SMD:R_2512_6332Metric
- added C27: 4.7nF, Capacitor_THT:C_Disc_D7.5mm_W5.0mm_P7.50mm, F.Cu at (110.2, 102.2)
- added C5: 10uF, Capacitor_SMD:C_0603_1608Metric, F.Cu at (66.6, 83.2)
- added NT1: NetTie, NetTie:NetTie-2_SMD_Pad2.0mm, F.Cu at (111.9, 78.0)
- added NT2: NetTie, NetTie:NetTie-2_SMD_Pad0.5mm, B.Cu at (107.2, 74.1)
- added R18: 47, Resistor_SMD:R_2512_6332Metric, F.Cu at (103.9, 82.9)
- C1, C25, C26, U1: moved to F.Cu
- C10: renamed from C27; moved to F.Cu
- C15: value 270UF -> 220UF; footprint PS:ALC80A271EB450 -> PS:CP_Radial_D18.0mm_P7.50mm
- C16: renamed from C17; moved to F.Cu
- C17: renamed from C18; moved to F.Cu
- C18: renamed from C19; moved to F.Cu
- C19: renamed from C20; moved to F.Cu
- C2: renamed from C3; moved to F.Cu
- C20: renamed from C16; value 10nF -> 1nF; footprint Capacitor_THT:C_Rect_L13.0mm_W4.0mm_P10.00mm_FKS3_FKP3_MKS4 -> Capacitor_THT:C_Disc_D7.5mm_W5.0mm_P7.50mm
- C3: renamed from C4; moved to F.Cu
- C4: renamed from C5; moved to F.Cu
- D1: renamed from D2; moved to F.Cu
- D2: renamed from D3; moved to F.Cu
- D3: renamed from D4; moved to F.Cu
- D6: renamed from D7; value S3MB-13-F -> STTH2R06U; moved to F.Cu
- R1: renamed from R2; moved to F.Cu
- R10: renamed from R13; moved to F.Cu
- R14: renamed from R18; value 649 -> 1.5k
- R15: renamed from R19; value 35.7k -> 35.2k
- R17: renamed from R21; moved to F.Cu
- R2: renamed from R3; moved to F.Cu
- R3: renamed from R5; footprint Resistor_SMD:R_0805_2012Metric_Pad1.20x1.40mm_HandSolder -> Resistor_SMD:R_0603_1608Metric; moved to F.Cu
- R4: renamed from R7; moved to F.Cu
- R5: renamed from R8; moved to F.Cu
- R6: renamed from R4; moved to F.Cu
- R7: renamed from R6; moved to F.Cu
- R8: renamed from R11; moved to F.Cu
- R9: renamed from R12; moved to F.Cu
- moved R4 51.6 mm to (92.2, 96.8), turned to 90 degrees
- moved HS1 41.7 mm to (82.5, 106.7), turned to 90 degrees
- moved C10 40.0 mm to (53.1, 86.9)
- moved C20 39.3 mm to (97.2, 89.2), turned to 90 degrees
- moved C1 38.3 mm to (58.5, 81.8), turned to 0 degrees
- moved C2 35.8 mm to (56.1, 86.9)
- moved D6 35.8 mm to (92.2, 86.2), turned to -90 degrees
- moved R17 34.7 mm to (103.9, 87.9), turned to 0 degrees
- moved C18 33.9 mm to (103.7, 130.4), turned to -90 degrees
- moved D7 28.2 mm to (74.7, 116.3), turned to -90 degrees
- moved U1 27.3 mm to (60.8, 85.5), turned to 0 degrees
- moved C4 26.4 mm to (66.7, 84.7)
- moved C17 25.9 mm to (101.6, 130.4), turned to 90 degrees
- moved D2 25.5 mm to (52.1, 81.9)
- moved R8 25.3 mm to (45.8, 81.9)
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- renumbered C10 to C11, D5 to D4, D6 to D5, D1 to D7, R15 to R11, R16 to R12, R17 to R13, R20 to R16
Connections:
- C1 pad 2: DCR_GND -> GND_DC_S
- C10 pad 1: DCR_GND -> GND_DC_S
- C16 pad 1: /PS/24V_O -> /PS/24V_F
- C16 pad 2: /PS/TR_OUT_GND -> OUT_GND
- C17 pad 1: /PS/TR_OUT_GND -> OUT_GND
- C17 pad 2: /PS/24V_O -> /PS/24V_F
- C18 pad 1: /PS/24V_O -> /PS/24V_F
- C18 pad 2: /PS/TR_OUT_GND -> OUT_GND
- C19 pad 1: /PS/TR_OUT_GND -> OUT_GND
- C19 pad 2: /PS/24V_O -> /PS/24V_F
- C2 pad 2: DCR_GND -> GND_DC_S
- C20 pad 1: Net-(D7-K) -> Net-(D6-K)
- C20 pad 2: /PS/AC_R_O -> Net-(C20-Pad2)
- C21 pad 1: /PS/24V_O -> /PS/24V_F
- C21 pad 2: /PS/TR_OUT_GND -> OUT_GND
- C22 pad 1: /PS/24V_O -> /PS/24V_F
- C22 pad 2: /PS/TR_OUT_GND -> OUT_GND
- C3 pad 2: DCR_GND -> GND_DC_P
- C4 pad 2: DCR_GND -> GND_DC_P
- C6 pad 2: DCR_GND -> GND_DC_P
- D6 pad 1: Net-(D7-K) -> Net-(D6-K)
- D7 pad 1: Net-(D1A-A) -> Net-(D7A-A)
- D7 pad 3: Net-(D1A-A) -> Net-(D7A-A)
- J2 pad 3: /PS/24V_O -> /PS/24V_F
- J2 pad 4: /PS/24V_O -> /PS/24V_F
- L1 pad 1: /PS/TR_OUT_GND -> /PS/24V_F
- L1 pad 2: OUT_GND -> /PS/24V_O
- R10 pad 2: DCR_GND -> GND_DC_S
- R17 pad 1: /PS/AC_R_O -> Net-(D6-K)
- R17 pad 2: Net-(D7-K) -> /PS/AC_R_O
- R3 pad 2: DCR_GND -> GND_DC_P
- R4 pad 2: DCR_GND -> GND_DC_P
- TR1 pad 1: /PS/AC_R_O -> /PS/TR_SW
- TR1 pad 11: Net-(D1A-A) -> OUT_GND
- TR1 pad 3: /PS/TR_SW -> /PS/AC_R_O
- TR1 pad 4: /PS/AUX -> DCR_GND
- TR1 pad 5: DCR_GND -> /PS/AUX
- TR1 pad 8: /PS/TR_OUT_GND -> Net-(D7A-A)
- U1 pad 4: DCR_GND -> GND_DC_S
- U2 pad 4: DCR_GND -> GND_DC_S
Routing:
- net GND_DC_S: track 0.00 -> 116.5 mm, vias 0 -> 2
- net /PS/AC_R_O: track 0.00 -> 113.7 mm
- net /PS/MOS_S: track 109.7 -> 3.72 mm
- net OUT_GND: track 18.7 -> 73.4 mm, vias 1 -> 2
- net DCR_GND: track 32.9 -> 82.5 mm, vias 2 -> 0
- net GND_DC_P: track 0.00 -> 49.5 mm, vias 0 -> 7
- net /PS/OPT_C: track 29.5 -> 73.2 mm
- net Net-(Q1-S): track 4.14 -> 36.3 mm, vias 0 -> 5
- net Net-(U1-OVP): track 32.7 -> 6.87 mm
- net /PS/TR_GAT: track 28.0 -> 3.77 mm, vias 2 -> 0
- net /PS/AUX: track 10.4 -> 28.4 mm
- net Net-(D6-K): track 0.00 -> 12.3 mm
- net Net-(D3-K): track 28.4 -> 37.3 mm, vias 0 -> 1
- net /PS/24V_F: track 0.00 -> 8.21 mm
- net Net-(U1-SS): track 7.14 -> 2.27 mm
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- added copper zone on B.Cu, net /PS/24V_F
- added copper zone on F.Cu, net /PS/24V_F
- added copper zone on B.Cu, net /PS/AC_R_I_2
- added copper zone on B.Cu, net GND_DC_P
- added copper zone on F.Cu, net GND_DC_P
- added copper zone on F.Cu, net GND_DC_S
- added copper zone on F.Cu, net Net-(D7A-A)
- removed copper zone on B.Cu, net /PS/AC_R_O
- removed copper zone on B.Cu, net /PS/TR_OUT_GND
- removed copper zone on F.Cu, net /PS/TR_OUT_GND
- removed copper zone on B.Cu, net Net-(D1A-A)
- removed copper zone on F.Cu, net Net-(D1A-A)
- removed copper zone on B.Cu, net Net-(D7-K)
Other:
- outline, holes or cut-outs redrawn
- board text added: "0.1500 mm / 0.1500 mm"
- board text added: "85.1000 mm x 120.1000 mm"
- board text added: "Dielectric"
- board text removed: "0.2000 mm / 0.0000 mm"
- board text removed: "85.0000 mm x 140.0000 mm"
- board text removed: "Dielectric 1"
