File: 01_ECAD/ACDC150V24.kicad_sch (KiCad schematic)
At the start: 0 parts

Commit message: Regular Update.
Other:
- note added: "120 MM"
- note removed: "140 MM"
- note removed: "5"
- note removed: "M3"
