File: 01_ECAD/PS.kicad_sch (KiCad schematic)
At the start: 73 parts, among them J1 B2P3-VH(LF)(SN), J2 B4P-VH(LF)(SN), Q1 IXFH20N100P, SW1 NE18 2A EE 6AMP, U1 UCC28600, U2 CNY17-1, U3 TL431DBZ

Commit message: UPDATE!
Parts:
- removed R1: 16.3K, Resistor_SMD:R_0805_2012Metric_Pad1.20x1.40mm_HandSolder, symbol Device:R_Small_US
- removed R22, R23, R24, R25, R26: 20K, Resistor_SMD:R_2512_6332Metric, symbol Device:R_Small_US
- added C27: 4.7nF, Capacitor_THT:C_Disc_D7.5mm_W5.0mm_P7.50mm, symbol ps:C_Small
- added C5: 10uF, Capacitor_SMD:C_0603_1608Metric, symbol ps:C_Small
- added NT1: NetTie, NetTie:NetTie-2_SMD_Pad2.0mm, symbol Device:NetTie_2
- added NT2: NetTie, NetTie:NetTie-2_SMD_Pad0.5mm, symbol Device:NetTie_2
- added R18: 47, Resistor_SMD:R_2512_6332Metric, symbol Device:R_Small_US
- C15: value 270UF -> 220UF; footprint PS:ALC80A271EB450 -> PS:CP_Radial_D18.0mm_P7.50mm
- C20: renamed from C16; value 10nF -> 1nF; footprint Capacitor_THT:C_Rect_L13.0mm_W4.0mm_P10.00mm_FKS3_FKP3_MKS4 -> Capacitor_THT:C_Disc_D7.5mm_W5.0mm_P7.50mm
- D6: renamed from D7; value S3MB-13-F -> STTH2R06U
- R3: renamed from R5; footprint Resistor_SMD:R_0805_2012Metric_Pad1.20x1.40mm_HandSolder -> Resistor_SMD:R_0603_1608Metric
- renumbered C27 to C10, C10 to C11, C17 to C16, C18 to C17, C19 to C18, C20 to C19, C3 to C2, C4 to C3, C5 to C4, D2 to D1, D3 to D2, D4 to D3, D5 to D4, D6 to D5, D1 to D7, R2 to R1, R13 to R10, R15 to R11, R16 to R12, R17 to R13, R18 to R14, R19 to R15, R20 to R16, R21 to R17, R3 to R2, R7 to R4, R8 to R5, R4 to R6, R6 to R7, R11 to R8, R12 to R9
Connections:
- net 24V_O: now also L1.2; no longer C16.1, C17.2, C18.1, C19.2, C21.1, C22.1, J2.3 (Pin_3), J2.4 (Pin_4)
- net AC_R_O: now also R17.2, TR1.3, R18.2; no longer C20.2, R17.1, TR1.1
- net AUX: now also TR1.5; no longer TR1.4
- net DCR_GND: now also TR1.4, NT1.2, NT2.2; no longer C1.2, C10.1, C2.2, C3.2, C4.2, C6.2, R10.2, R3.2, R4.2, TR1.5, U1.4 (GND), U2.4
- net OUT_GND: now also C16.2, C17.1, C18.2, C19.1, C21.2, C22.2, TR1.11, C27.1; no longer L1.2
- net TR_SW: now also TR1.1; no longer TR1.3
- net at C20.1, D6.1 (K): now also R17.1; no longer R17.2
- net at C3.1, C4.1, D2.1 (K)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: now also C5.1
- net at D7.1 (A), D7.3 (K): now also TR1.8; no longer TR1.11
- removed net TR_OUT_GND: C16.2, C17.1, C18.2, C19.1, C21.2, C22.2, L1.1, TR1.8
- new net: C20.2, R18.1
- new net 24V_F: C16.1, C17.2, C18.1, C19.2, C21.1, C22.1, J2.3 (Pin_3), J2.4 (Pin_4), L1.1
- new net GND_DC_P: C27.2, C3.2, C4.2, C5.2, C6.2, NT1.1, R3.2, R4.2
- new net GND_DC_S: C1.2, C10.1, C2.2, NT2.1, R10.2, U1.4 (GND), U2.4
Other:
- note added: "STAR GROUND"
- moved on the sheet: C16, C17, C18, C19, C20, C21, C22, C6, D2, D6, D7A, D7B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

Commit message: Update.
Parts:
- removed D1: RB520SM-40T2R, Diode_SMD:D_SOD-523, symbol Device:D_Schottky
- added C28: 1nF, Capacitor_THT:C_Disc_D7.5mm_W5.0mm_P7.50mm, symbol ps:C_Small
- added D1: PMEG100T10ELXDX, Diode_SMD:D_SOD-323, symbol Diode:UF5407
- added HS2: V5629W220, PS:V5629W220, symbol Mechanical:Heatsink
- added R19: 4.3k, Resistor_SMD:R_0603_1608Metric, symbol Device:R_Small_US
- added R20: 47, Resistor_THT:R_Axial_DIN0516_L15.5mm_D5.0mm_P5.08mm_Vertical, symbol Device:R_Small_US
- D2, D3: value VS-2EMH01HM3/5AT -> PMEG100T10ELXDX; footprint Diode_SMD:D_SMA -> Diode_SMD:D_SOD-323
- R15: value 35.2k -> 4.3k; PN TNPW080535K2BEEN -> ERJ-PB3D4301V
- R16: value 4.12k -> 1k; PN ERJ-PB3B4121V -> ERJ-PB3D1001V
- R17, R18: footprint Resistor_SMD:R_2512_6332Metric -> Resistor_THT:R_Axial_DIN0516_L15.5mm_D5.0mm_P5.08mm_Vertical
- R8: footprint Resistor_SMD:R_1206_3216Metric_Pad1.30x1.75mm_HandSolder -> Resistor_SMD:R_0603_1608Metric; PN (none) -> ERJ-PA3F20R0V
Connections:
- net 24V_F: now also R14.2, R15.2
- net 24V_O: now also R20.2; no longer R14.2, R15.2
- net TR_GAT: now also D1.1 (K)
- net at Q1.1 (G), R1.1, R3.1: now also D1.2 (A)
- net at C3.1, C4.1, C5.1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: now also R8.2; no longer D2.1 (K)
- net at D7.1 (A), D7.3 (K), TR1.8: now also C28.2
- net at C6.1, D3.1 (K): now also D2.2 (A); no longer R8.1
- net at C13.2, C14.2, R16.2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: now also R19.1; no longer R15.1
- new net: D2.1 (K), R8.1
- new net: R15.1, R19.2
- new net: C28.1, R20.1
Other:
- moved on the sheet: R15, R8

Commit message: Adding To-Do.txt , First initial working Design.
Parts:
- C13: value 43pF -> 68pF; PN GRM1885C1H430JA01D -> 0603N680J500CT
- C14: value 27nF -> 56nF; PN (none) -> 0603B563K500CT
- R11: value 1K -> 499; PN MR06X1001FTL -> RN73R1JTTD4990B25
- R13: value 93.1k -> 48.7K; PN RK73H1JTTDD9312F -> ERJ-PB3B4872V
- R15: value 4.3k -> 36K; PN ERJ-PB3D4301V -> ERJ-PB3B3602V
- R16: value 1k -> 4.3K; PN ERJ-PB3D1001V -> ERJ-PB3B4301V
- R19: value 4.3k -> 976; PN ERJ-PB3D4301V -> ERJ-PB3B9760V
Changed lines of the file:
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@@
       (effects (font (size 1.27 1.27)) (justify left))
     )
-    (property "Value" "93.1k" (at 180.34 213.36 0)
+    (property "Value" "48.7K" (at 180.34 213.36 0)
       (effects (font (size 1.27 1.27)) (justify left))
     )
@@
       (effects (font (size 1.27 1.27)) hide)
     )
-    (property "PN" "RK73H1JTTDD9312F" (at 177.8 213.36 0)
+    (property "PN" "ERJ-PB3B4872V" (at 177.8 213.36 0)
       (effects (font (size 1.27 1.27)) hide)
     )
@@
       (effects (font (size 1.27 1.27)) (justify left))
     )
-    (property "Value" "27nF" (at 190.5 211.455 0) (do_not_autoplace)
+    (property "Value" "56nF" (at 190.5 211.455 0) (do_not_autoplace)
       (effects (font (size 1.27 1.27)) (justify left))
     )
@@
       (effects (font (size 1.27 1.27)) (justify left))
     )
-    (property "PN" "" (at 190.5 213.36 0)
+    (property "PN" "0603B563K500CT" (at 190.5 213.36 0)
       (effects (font (size 1.27 1.27)) hide)
     )
@@
       (effects (font (size 1.27 1.27)) (justify left))
     )
-    (property "Value" "1K" (at 167.64 193.04 0)
+    (property "Value" "499" (at 167.64 193.04 0)
       (effects (font (size 1.27 1.27)) (justify left))
     )
@@
       (effects (font (size 1.27 1.27)) hide)
     )
-    (property "PN" "MR06X1001FTL" (at 167.64 190.5 0)
+    (property "PN" "RN73R1JTTD4990B25" (at 167.64 190.5 0)
       (effects (font (size 1.27 1.27)) hide)
     )
@@
       (effects (font (size 1.27 1.27)) (justify left))
     )
-    (property "Value" "43pF" (at 185.42 201.295 0) (do_not_autoplace)
+    (property "Value" "68pF" (at 185.42 201.295 0) (do_not_autoplace)
       (effects (font (size 1.27 1.27)) (justify left))
     )
@@
       (effects (font (size 1.27 1.27)) (justify left))
     )
-    (property "PN" "GRM1885C1H430JA01D" (at 185.42 203.2 0)
+    (property "PN" "0603N680J500CT" (at 185.42 203.2 0)
       (effects (font (size 1.27 1.27)) hide)
     )
@@
       (effects (font (size 1.27 1.27)) (justify left))
     )
-    (property "Value" "4.3k" (at 200.66 203.2 0)
+    (property "Value" "976" (at 200.66 203.2 0)
       (effects (font (size 1.27 1.27)) (justify left))
     )
@@
       (effects (font (size 1.27 1.27)) hide)
     )
-    (property "PN" "ERJ-PB3D4301V" (at 200.66 200.66 0)
+    (property "PN" "ERJ-PB3B9760V" (at 200.66 200.66 0)
       (effects (font (size 1.27 1.27)) hide)
     )
@@
       (effects (font (size 1.27 1.27)) (justify left))
     )
-    (property "Value" "4.3k" (at 200.66 195.58 0)
+    (property "Value" "36K" (at 200.66 195.58 0)
       (effects (font (size 1.27 1.27)) (justify left))
     )
@@
       (effects (font (size 1.27 1.27)) hide)
     )
-    (property "PN" "ERJ-PB3D4301V" (at 200.66 193.04 0)
+    (property "PN" "ERJ-PB3B3602V" (at 200.66 193.04 0)
       (effects (font (size 1.27 1.27)) hide)
     )
@@
       (effects (font (size 1.27 1.27)) (justify left))
     )
-    (property "Value" "1k" (at 200.66 226.06 0)
+    (property "Value" "4.3K" (at 200.66 226.06 0)
       (effects (font (size 1.27 1.27)) (justify left))
     )
@@
       (effects (font (size 1.27 1.27)) hide)
     )
-    (property "PN" "ERJ-PB3D1001V" (at 200.66 223.52 0)
-      (effects (font (size 1.27 1.27)) hide)
-    )
+    (property "PN" "ERJ-PB3B4301V" (at 200.66 223.52 0)
+      (effects (font (size 1.27 1.27)) hide)
+    )
