File: 01_ECAD/ACDC120V24.kicad_pcb (KiCad board)
At the start: 2 copper layers, 85 x 120 mm, 81 parts, among them J1 B2P3-VH(LF)(SN), J2 B4P-VH(LF)(SN), Q1 SIHA6N80AE-GE3, SW1 NE18 2A EE 6AMP, U1 UCC28600, U2 CNY17-1, U3 TL431DBZ

Commit message: Update.
Parts:
- removed C19: 10nF, Capacitor_THT:C_Disc_D7.5mm_W5.0mm_P7.50mm
- removed R19, R20, R21: 47, Resistor_THT:R_Axial_DIN0516_L15.5mm_D5.0mm_P5.08mm_Vertical
- C22: value 10nF -> 4.7nF
- NT1: moved to B.Cu
- R10: value 86.6k -> 200k
- R11: value 31.875k -> 39k
- R22: value 20k -> 470
- R23: value 20k -> 10
- moved R22 123.8 mm to (58.7, 108.6), turned to 0 degrees
- moved D4 101.0 mm to (66.9, 110.8)
- moved R4 82.7 mm to (56.2, 104.1), turned to 0 degrees
- moved R3 80.5 mm to (56.2, 101.1), turned to 0 degrees
- moved R2 80.3 mm to (56.2, 102.6), turned to 0 degrees
- moved D7 77.8 mm to (51.4, 109.1), turned to 180 degrees
- moved D2 74.4 mm to (59.3, 100.9), turned to 0 degrees
- moved D1 74.1 mm to (59.3, 102.8), turned to 180 degrees
- moved R23 73.4 mm to (56.7, 97.0)
- moved R9 67.7 mm to (67.0, 107.4)
- moved C6 67.3 mm to (70.4, 109.3)
- moved C22 66.0 mm to (51.2, 104.8), turned to 90 degrees
- moved D3 65.7 mm to (67.0, 104.2), turned to -90 degrees
- moved C3 64.5 mm to (68.7, 104.2), turned to -90 degrees
- moved R5 64.3 mm to (48.7, 89.6)
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Connections:
- C12 pad 2: GND_DC_P -> DCR_GND
- C22 pad 1: Net-(C22-Pad1) -> Net-(D7-K)
- C22 pad 2: /PS/AC_R_O -> Net-(C22-Pad2)
- R23 pad 1: Net-(D7-K) -> Net-(C22-Pad2)
- R23 pad 2: Net-(C22-Pad1) -> /PS/AC_R_O
Routing:
- net /PS/AC_R_O: track 82.7 -> 19.3 mm, vias 3 -> 0
- net /PS/AUX: track 0.00 -> 52.3 mm
- net /PS/OPT_C: track 60.3 -> 18.3 mm
- net GND_DC_S: track 55.3 -> 13.6 mm, vias 2 -> 3
- net Net-(D3-K): track 11.4 -> 32.6 mm
- net OUT_GND: track 17.8 -> 5.08 mm, vias 5 -> 7
- net Net-(Q1-S): track 31.5 -> 21.7 mm, vias 1 -> 2
- net Net-(D7-K): track 0.86 -> 10.4 mm
- net /PS/TR_GAT: track 5.07 -> 13.1 mm, vias 0 -> 2
- net Net-(Q1-G): track 6.44 -> 14.3 mm
- net GND_DC_P: track 0.00 -> 7.03 mm, vias 6 -> 12
- net Net-(C22-Pad2): track 0.00 -> 5.40 mm
- net /PS/24V_F: track 9.12 -> 4.27 mm
- net Net-(U1-OVP): track 6.87 -> 3.59 mm
- net Net-(R7-Pad1): track 0.00 -> 2.90 mm
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- added copper zone on B.Cu, net /PS/TR_SW
- added copper zone on F.Cu, net /PS/TR_SW
- added copper zone on B.Cu, net GND_DC_P
- added copper zone on B.Cu, net GND_DC_S
- added copper zone on F.Cu, net Net-(Q1-S)
- removed copper zone on F.Cu, net (none)
- removed copper zone on B.Cu, net /PS/AC_R_O
- removed copper zone on F.Cu, net Net-(D3-K)
- removed copper zone on B.Cu, net Net-(D8A-A)
Other:
- board size 85 x 120 mm -> 85 x 128.5 mm
- board text added: "85.0000 mm x 128.5000 mm"
- board text removed: "85.1000 mm x 120.1000 mm"
